File: sch/UARTtoBluetoothSerial/UARTtoBluetoothSerial.sch (KiCad schematic (older format))
At the start: 15 parts, among them IC1 NJM12888F33-TE1, J1 UART, SW1 SSSS213202, U1 ESP32-WROOM-32

Commit message: kicadライブラリのpath調整
Parts:
- IC1: symbol NJM12888F33-TE1:NJM12888F33-TE1 -> UARTtoBluetoothSerial-rescue:NJM12888F33-TE1-NJM12888F33-TE1
- S2, S3: symbol SKRPACE010:SKRPACE010 -> UARTtoBluetoothSerial-rescue:SKRPACE010-SKRPACE010
Changed lines of the file:
@@
 	5300 5250 5300 5350
 $Comp
-L SKRPACE010:SKRPACE010 S3
+L UARTtoBluetoothSerial-rescue:SKRPACE010-SKRPACE010 S3
 U 1 1 5F89BCE7
 P 10000 4650
@@
 	9300 5100 9300 5200
 $Comp
-L SKRPACE010:SKRPACE010 S2
+L UARTtoBluetoothSerial-rescue:SKRPACE010-SKRPACE010 S2
 U 1 1 5F92BA1B
 P 9950 3050
@@
 LED
 $Comp
-L NJM12888F33-TE1:NJM12888F33-TE1 IC1
+L UARTtoBluetoothSerial-rescue:NJM12888F33-TE1-NJM12888F33-TE1 IC1
 U 1 1 5F8DACE8
 P 2100 4050

Commit message: 回路図修正
Parts:
- R1: value 100 -> 10k
Changed lines of the file:
@@
 P 7450 2700
 F 0 "R1" H 7380 2654 50  0000 R CNN
-F 1 "100" H 7380 2745 50  0000 R CNN
+F 1 "10k" H 7380 2745 50  0000 R CNN
 F 2 "Resistor_SMD:R_0603_1608Metric" V 7380 2700 50  0001 C CNN
 F 3 "~" H 7450 2700 50  0001 C CNN
